File: led_unterm_bett.sch (KiCad schematic (older format))
At the start: 27 parts, among them J1 Conn_01x03, J2 Conn_01x03, J3 Conn_01x03, J4 Conn_01x02, J5 Barrel_Jack, J6 Conn_01x04, Q1 BSS138, Q2 BSS138, Q3 BSS138, U1 NodeMCU1.0(ESP-12E), U2 LM7805_TO220

Commit message: finish schematic and devise netlist
ready start routing
Parts:
- removed J5: Barrel_Jack, symbol Barrel_Jack
- added J5: Screw_Terminal_01x02, TerminalBlock:TerminalBlock_bornier-2_P5.08mm, symbol Screw_Terminal_01x02
- C1, C2, C3, C4, C5: footprint (none) -> Capacitors_SMD:C_0805_HandSoldering
- C6, C7, C8: footprint (none) -> Capacitors_THT:CP_Radial_D10.0mm_P3.50mm
- D1, D2, D3: footprint (none) -> Diodes_SMD:D_MiniMELF_Handsoldering
- J1, J3: footprint (none) -> Pin_Headers:Pin_Header_Straight_1x03_Pitch1.00mm_SMD_Pin1Left
- J2: footprint (none) -> Pin_Headers:Pin_Header_Straight_1x03_Pitch1.00mm_SMD_Pin1Right
- J4: footprint (none) -> Pin_Headers:Pin_Header_Straight_1x02_Pitch1.27mm_SMD_Pin1Right
- J6: footprint (none) -> Pin_Headers:Pin_Header_Straight_1x04_Pitch2.54mm_SMD_Pin1Right
- R1: value 86k -> 11k; footprint (none) -> Resistors_SMD:R_0805_HandSoldering
- R2, R3, R4, R5: footprint (none) -> Resistors_SMD:R_0805_HandSoldering
- U1: footprint (none) -> ESP8266:NodeMCU1.0(12-E)
- U2: footprint TO_SOT_Packages_THT:TO-220_Vertical -> TO_SOT_Packages_THT:TO-220-3_Vertical
Connections:
- net +12V: now also J5.2 (Pin_2); no longer J1.3 (Pin_3), J2.3 (Pin_3), J3.3 (Pin_3)
- net +5V: now also J1.3 (Pin_3), J2.3 (Pin_3), J3.3 (Pin_3)
- net GND: now also J5.1 (Pin_1)
Changed lines of the file:
@@
 F 0 "U1" H 4850 3300 60  0000 C CNN
 F 1 "NodeMCU1.0(ESP-12E)" H 4850 1600 60  0000 C CNN
-F 2 "" H 4250 1600 60  0000 C CNN
+F 2 "ESP8266:NodeMCU1.0(12-E)" H 4250 1600 60  0001 C CNN
 F 3 "" H 4250 1600 60  0000 C CNN
 	1    4850 2450
@@
 F 0 "R3" V 8380 1400 50  0000 C CNN
 F 1 "100k" V 8300 1400 50  0000 C CNN
-F 2 "" V 8230 1400 50  0001 C CNN
+F 2 "Resistors_SMD:R_0805_HandSoldering" V 8230 1400 50  0001 C CNN
 F 3 "" H 8300 1400 50  0001 C CNN
 	1    8300 1400
@@
 F 0 "R4" V 8380 2200 50  0000 C CNN
 F 1 "100k" V 8300 2200 50  0000 C CNN
-F 2 "" V 8230 2200 50  0001 C CNN
+F 2 "Resistors_SMD:R_0805_HandSoldering" V 8230 2200 50  0001 C CNN
 F 3 "" H 8300 2200 50  0001 C CNN
 	1    8300 2200
@@
 F 0 "R5" V 8380 3000 50  0000 C CNN
 F 1 "100k" V 8300 3000 50  0000 C CNN
-F 2 "" V 8230 3000 50  0001 C CNN
+F 2 "Resistors_SMD:R_0805_HandSoldering" V 8230 3000 50  0001 C CNN
 F 3 "" H 8300 3000 50  0001 C CNN
 	1    8300 3000
@@
 F 0 "J6" H 9550 1250 50  0000 C CNN
 F 1 "Conn_01x04" H 9550 750 50  0000 C CNN
-F 2 "" H 9550 1050 50  0001 C CNN
+F 2 "Pin_Headers:Pin_Header_Straight_1x04_Pitch2.54mm_SMD_Pin1Right" H 9550 1050 50  0001 C CNN
 F 3 "" H 9550 1050 50  0001 C CNN
 	1    9550 1050
@@
 $EndComp
 $Comp
-L Barrel_Jack J5
-U 1 1 5F551C69
-P 6600 4600
-F 0 "J5" H 6600 4810 50  0000 C CNN
-F 1 "Barrel_Jack" H 6600 4425 50  0000 C CNN
-F 2 "" H 6650 4560 50  0001 C CNN
-F 3 "" H 6650 4560 50  0001 C CNN
-	1    6600 4600
-	1    0    0    -1
-$EndComp
-$Comp
 L +12V #PWR09
 U 1 1 5F551D85
@@
 F 0 "U2" H 8350 4625 50  0000 C CNN
 F 1 "LM7805_TO220" H 8500 4625 50  0000 L CNN
-F 2 "TO_SOT_Packages_THT:TO-220_Vertical" H 8500 4725 50  0001 C CIN
+F 2 "TO_SOT_Packages_THT:TO-220-3_Vertical" H 8500 4725 50  0001 C CIN
 F 3 "" H 8500 4450 50  0001 C CNN
 	1    8500 4500
@@
 F 0 "C6" H 7875 4750 50  0000 L CNN
 F 1 "10u" H 7875 4550 50  0000 L CNN
-F 2 "" H 7888 4500 50  0001 C CNN
+F 2 "Capacitors_THT:CP_Radial_D10.0mm_P3.50mm" H 7888 4500 50  0001 C CNN
 F 3 "" H 7850 4650 50  0001 C CNN
 	1    7850 4650
@@
 F 0 "C7" H 9175 4750 50  0000 L CNN
 F 1 "10u" H 9175 4550 50  0000 L CNN
-F 2 "" H 9188 4500 50  0001 C CNN
+F 2 "Capacitors_THT:CP_Radial_D10.0mm_P3.50mm" H 9188 4500 50  0001 C CNN
 F 3 "" H 9150 4650 50  0001 C CNN
 	1    9150 4650
@@
 F 0 "J4" H 3950 3450 50  0000 C CNN
 F 1 "Conn_01x02" H 3950 3150 50  0000 C CNN
-F 2 "" H 3950 3350 50  0001 C CNN
+F 2 "Pin_Headers:Pin_Header_Straight_1x02_Pitch1.27mm_SMD_Pin1Right" H 3950 3350 50  0001 C CNN
 F 3 "" H 3950 3350 50  0001 C CNN
 	1    3950 3350
@@
 F 0 "C3" H 4075 3700 50  0000 L CNN
 F 1 "100n" H 4075 3500 50  0000 L CNN
-F 2 "" H 4088 3450 50  0001 C CNN
+F 2 "Capacitors_SMD:C_0805_HandSoldering" H 4088 3450 50  0001 C CNN
 F 3 "" H 4050 3600 50  0001 C CNN
 	1    4050 3600
@@
 F 0 "C5" H 6075 3250 50  0000 L CNN
 F 1 "100n" H 6075 3050 50  0000 L CNN
-F 2 "" H 6088 3000 50  0001 C CNN
+F 2 "Capacitors_SMD:C_0805_HandSoldering" H 6088 3000 50  0001 C CNN
 F 3 "" H 6050 3150 50  0001 C CNN
 	1    6050 3150
@@
 F 0 "C4" H 6075 2350 50  0000 L CNN
 F 1 "100n" H 6075 2150 50  0000 L CNN
-F 2 "" H 6088 2100 50  0001 C CNN
+F 2 "Capacitors_SMD:C_0805_HandSoldering" H 6088 2100 50  0001 C CNN
 F 3 "" H 6050 2250 50  0001 C CNN
 	1    6050 2250
@@
 F 0 "C2" H 3675 2850 50  0000 L CNN
 F 1 "100n" H 3675 2650 50  0000 L CNN
-F 2 "" H 3688 2600 50  0001 C CNN
+F 2 "Capacitors_SMD:C_0805_HandSoldering" H 3688 2600 50  0001 C CNN
 F 3 "" H 3650 2750 50  0001 C CNN
 	1    3650 2750
@@
 F 0 "J1" H 1300 950 50  0000 C CNN
 F 1 "Conn_01x03" H 1300 550 50  0000 C CNN
-F 2 "" H 1300 750 50  0001 C CNN
+F 2 "Pin_Headers:Pin_Header_Straight_1x03_Pitch1.00mm_SMD_Pin1Left" H 1300 750 50  0001 C CNN
 F 3 "" H 1300 750 50  0001 C CNN
 	1    1300 750
@@
 F 0 "J2" H 1300 1550 50  0000 C CNN
 F 1 "Conn_01x03" H 1300 1150 50  0000 C CNN
-F 2 "" H 1300 1350 50  0001 C CNN
+F 2 "Pin_Headers:Pin_Header_Straight_1x03_Pitch1.00mm_SMD_Pin1Right" H 1300 1350 50  0001 C CNN
 F 3 "" H 1300 1350 50  0001 C CNN
 	1    1300 1350
@@
 F 0 "J3" H 1300 2100 50  0000 C CNN
 F 1 "Conn_01x03" H 1300 1700 50  0000 C CNN
-F 2 "" H 1300 1900 50  0001 C CNN
+F 2 "Pin_Headers:Pin_Header_Straight_1x03_Pitch1.00mm_SMD_Pin1Left" H 1300 1900 50  0001 C CNN
 F 3 "" H 1300 1900 50  0001 C CNN
 	1    1300 1900
@@
 $EndComp
 $Comp
-L +12V #PWR017
-U 1 1 5F56341E
-P 1500 650
-F 0 "#PWR017" H 1500 500 50  0001 C CNN
-F 1 "+12V" H 1500 790 50  0000 C CNN
-F 2 "" H 1500 650 50  0001 C CNN
-F 3 "" H 1500 650 50  0001 C CNN
-	1    1500 650
-	1    0    0    -1
-$EndComp
-$Comp
-L +12V #PWR018
-U 1 1 5F56345A
-P 1500 1250
-F 0 "#PWR018" H 1500 1100 50  0001 C CNN
-F 1 "+12V" H 1500 1390 50  0000 C CNN
-F 2 "" H 1500 1250 50  0001 C CNN
-F 3 "" H 1500 1250 50  0001 C CNN
-	1    1500 1250
-	1    0    0    -1
-$EndComp
-$Comp
-L +12V #PWR019
-U 1 1 5F563496
-P 1500 1800
-F 0 "#PWR019" H 1500 1650 50  0001 C CNN
-F 1 "+12V" H 1500 1940 50  0000 C CNN
-F 2 "" H 1500 1800 50  0001 C CNN
-F 3 "" H 1500 1800 50  0001 C CNN
-	1    1500 1800
-	1    0    0    -1
-$EndComp
-$Comp
 L D D2
 U 1 1 5F5637F2
@@
 F 0 "D2" H 1850 1450 50  0000 C CNN
 F 1 "D" H 1850 1250 50  0000 C CNN
-F 2 "" H 1850 1350 50  0001 C CNN
+F 2 "Diodes_SMD:D_MiniMELF_Handsoldering" H 1850 1350 50  0001 C CNN
 F 3 "" H 1850 1350 50  0001 C CNN
 	1    1850 1350
@@
 F 0 "D3" H 1850 2000 50  0000 C CNN
 F 1 "D" H 1850 1800 50  0000 C CNN
-F 2 "" H 1850 1900 50  0001 C CNN
+F 2 "Diodes_SMD:D_MiniMELF_Handsoldering" H 1850 1900 50  0001 C CNN
 F 3 "" H 1850 1900 50  0001 C CNN
 	1    1850 1900
@@
 F 0 "D1" H 1850 850 50  0000 C CNN
 F 1 "D" H 1850 650 50  0000 C CNN
-F 2 "" H 1850 750 50  0001 C CNN
+F 2 "Diodes_SMD:D_MiniMELF_Handsoldering" H 1850 750 50  0001 C CNN
 F 3 "" H 1850 750 50  0001 C CNN
 	1    1850 750
@@
 P 2550 1500
 F 0 "R1" V 2630 1500 50  0000 C CNN
-F 1 "86k" V 2550 1500 50  0000 C CNN
-F 2 "" V 2480 1500 50  0001 C CNN
+F 1 "11k" V 2550 1500 50  0000 C CNN
+F 2 "Resistors_SMD:R_0805_HandSoldering" V 2480 1500 50  0001 C CNN
 F 3 "" H 2550 1500 50  0001 C CNN
 	1    2550 1500
@@
 F 0 "R2" V 2630 1800 50  0000 C CNN
 F 1 "33k" V 2550 1800 50  0000 C CNN
-F 2 "" V 2480 1800 50  0001 C CNN
+F 2 "Resistors_SMD:R_0805_HandSoldering" V 2480 1800 50  0001 C CNN
 F 3 "" H 2550 1800 50  0001 C CNN
 	1    2550 1800
@@
 $EndComp
 $Comp
-L GND #PWR020
+L GND #PWR017
 U 1 1 5F563C1D
 P 2550 1950
-F 0 "#PWR020" H 2550 1700 50  0001 C CNN
+F 0 "#PWR017" H 2550 1700 50  0001 C CNN
 F 1 "GND" H 2550 1800 50  0000 C CNN
 F 2 "" H 2550 1950 50  0001 C CNN
@@
 F 0 "C1" H 3075 1900 50  0000 L CNN
 F 1 "100n" H 3075 1700 50  0000 L CNN
-F 2 "" H 3088 1650 50  0001 C CNN
+F 2 "Capacitors_SMD:C_0805_HandSoldering" H 3088 1650 50  0001 C CNN
 F 3 "" H 3050 1800 50  0001 C CNN
 	1    3050 1800
@@
 F 0 "C8" H 3275 2950 50  0000 L CNN
 F 1 "1u" H 3275 2750 50  0000 L CNN
-F 2 "" H 3288 2700 50  0001 C CNN
+F 2 "Capacitors_THT:CP_Radial_D10.0mm_P3.50mm" H 3288 2700 50  0001 C CNN
 F 3 "" H 3250 2850 50  0001 C CNN
 	1    3250 2850
@@
 	3100 2850 3100 2650
 Connection ~ 3100 2650
+$Comp
+L +5V #PWR018
+U 1 1 5FD4F943
+P 1500 650
+F 0 "#PWR018" H 1500 500 50  0001 C CNN
+F 1 "+5V" H 1500 790 50  0000 C CNN
+F 2 "" H 1500 650 50  0001 C CNN
+F 3 "" H 1500 650 50  0001 C CNN
+	1    1500 650
+	1    0    0    -1
+$EndComp
+$Comp
+L +5V #PWR019
+U 1 1 5FD4FC42
+P 1500 1250
+F 0 "#PWR019" H 1500 1100 50  0001 C CNN
+F 1 "+5V" H 1500 1390 50  0000 C CNN
+F 2 "" H 1500 1250 50  0001 C CNN
+F 3 "" H 1500 1250 50  0001 C CNN
+	1    1500 1250
+	1    0    0    -1
+$EndComp
+$Comp
+L +5V #PWR020
+U 1 1 5FD4FC9E
+P 1500 1800
+F 0 "#PWR020" H 1500 1650 50  0001 C CNN
+F 1 "+5V" H 1500 1940 50  0000 C CNN
+F 2 "" H 1500 1800 50  0001 C CNN
+F 3 "" H 1500 1800 50  0001 C CNN
+	1    1500 1800
+	1    0    0    -1
+$EndComp
+$Comp
+L Screw_Terminal_01x02 J5
+U 1 1 5FD50EFF
+P 6700 4600
+F 0 "J5" H 6700 4700 50  0000 C CNN
+F 1 "Screw_Terminal_01x02" H 6700 4400 50  0000 C CNN
+F 2 "TerminalBlock:TerminalBlock_bornier-2_P5.08mm" H 6700 4600 50  0001 C CNN
+F 3 "" H 6700 4600 50  0001 C CNN
+	1    6700 4600
+	-1   0    0    1
+$EndComp
 $EndSCHEMATC

Commit message: placement complete
Parts:
- J1, J3: footprint Pin_Headers:Pin_Header_Straight_1x03_Pitch1.00mm_SMD_Pin1Left -> Pin_Headers:Pin_Header_Straight_1x03_Pitch2.54mm
- J2: footprint Pin_Headers:Pin_Header_Straight_1x03_Pitch1.00mm_SMD_Pin1Right -> Pin_Headers:Pin_Header_Straight_1x03_Pitch2.54mm
- J4: footprint Pin_Headers:Pin_Header_Straight_1x02_Pitch1.27mm_SMD_Pin1Right -> Pin_Headers:Pin_Header_Straight_1x02_Pitch2.54mm
- J6: footprint Pin_Headers:Pin_Header_Straight_1x04_Pitch2.54mm_SMD_Pin1Right -> Pin_Headers:Pin_Header_Straight_1x04_Pitch2.54mm
Connections:
- net +12V: now also J6.4 (Pin_4); no longer J6.1 (Pin_1)
- net +5V: now also J1.2 (Pin_2), J2.2 (Pin_2), J3.2 (Pin_2); no longer J1.3 (Pin_3), J2.3 (Pin_3), J3.3 (Pin_3)
- net GND: now also J1.3 (Pin_3), J2.3 (Pin_3), J3.3 (Pin_3); no longer J1.1 (Pin_1), J2.1 (Pin_1), J3.1 (Pin_1)
- net at Q1.3 (D): now also J6.1 (Pin_1); no longer J6.2 (Pin_2)
- net at Q2.3 (D): now also J6.2 (Pin_2); no longer J6.3 (Pin_3)
- net at Q3.3 (D): now also J6.3 (Pin_3); no longer J6.4 (Pin_4)
- net at D1.2 (A): now also J1.1 (Pin_1); no longer J1.2 (Pin_2)
- net at D2.2 (A): now also J2.1 (Pin_1); no longer J2.2 (Pin_2)
- net at D3.2 (A): now also J3.1 (Pin_1); no longer J3.2 (Pin_2)
Other:
- moved on the sheet: D1, D2, D3

Commit message: finish routing for etched PCB
Parts:
- U1: footprint ESP8266:NodeMCU1.0(12-E) -> ESP8266:ESP12F-Devkit-V3
Changed lines of the file:
@@
 F 0 "U1" H 4850 3300 60  0000 C CNN
 F 1 "NodeMCU1.0(ESP-12E)" H 4850 1600 60  0000 C CNN
-F 2 "ESP8266:NodeMCU1.0(12-E)" H 4250 1600 60  0001 C CNN
+F 2 "ESP8266:ESP12F-Devkit-V3" H 4250 1600 60  0001 C CNN
 F 3 "" H 4250 1600 60  0000 C CNN
 	1    4850 2450

Commit message: kicad 4->5, jlcpcb drc
Load design rules from https://github.com/sethhillbrand/kicad_templates.
Used rules for jlcpcb.com
Parts:
- C1, C2, C3, C4, C5: symbol C -> Device:C
- C6, C7, C8: symbol CP -> Device:CP
- D1, D2, D3: symbol D -> Device:D
- J1, J2, J3: symbol Conn_01x03 -> conn:Conn_01x03
- J4: symbol Conn_01x02 -> conn:Conn_01x02
- J5: symbol Screw_Terminal_01x02 -> conn:Screw_Terminal_01x02
- J6: symbol Conn_01x04 -> conn:Conn_01x04
- Q1, Q2, Q3: symbol BSS138 -> transistors:BSS138
- R1, R2, R3, R4, R5: symbol R -> Device:R
- U1: symbol NodeMCU1.0(ESP-12E) -> ESP8266:NodeMCU1.0(ESP-12E)
- U2: symbol LM7805_TO220 -> regul:LM7805_TO220
Changed lines of the file:
@@
-EESchema Schematic File Version 2
-LIBS:power
-LIBS:device
-LIBS:switches
-LIBS:relays
-LIBS:motors
-LIBS:transistors
-LIBS:conn
-LIBS:linear
-LIBS:regul
-LIBS:74xx
-LIBS:cmos4000
-LIBS:adc-dac
-LIBS:memory
-LIBS:xilinx
-LIBS:microcontrollers
-LIBS:dsp
-LIBS:microchip
-LIBS:analog_switches
-LIBS:motorola
-LIBS:texas
-LIBS:intel
-LIBS:audio
-LIBS:interface
-LIBS:digital-audio
-LIBS:philips
-LIBS:display
-LIBS:cypress
-LIBS:siliconi
-LIBS:opto
-LIBS:atmel
-LIBS:contrib
-LIBS:valves
-LIBS:ESP8266
-LIBS:led_unterm_bett-cache
-EELAYER 25 0
+EESchema Schematic File Version 4
+EELAYER 30 0
 EELAYER END
 $Descr A4 11693 8268
@@
 $EndDescr
 $Comp
-L NodeMCU1.0(ESP-12E) U1
+L ESP8266:NodeMCU1.0(ESP-12E) U1
 U 1 1 5F55090F
 P 4850 2450
@@
 $EndComp
 $Comp
-L GND #PWR01
+L power:GND #PWR01
 U 1 1 5F5509D5
 P 3950 3050
@@
 $EndComp
 $Comp
-L GND #PWR02
+L power:GND #PWR02
 U 1 1 5F550A24
 P 3000 2650
@@
 $EndComp
 $Comp
-L GND #PWR03
+L power:GND #PWR03
 U 1 1 5F550A32
 P 6200 2350
@@
 $EndComp
 $Comp
-L GND #PWR04
+L power:GND #PWR04
 U 1 1 5F550A40
 P 6300 3050
@@
 $EndComp
 $Comp
-L BSS138 Q1
+L transistors:BSS138 Q1
 U 1 1 5F550A7E
 P 8650 1250
@@
 $EndComp
 $Comp
-L R R3
+L Device:R R3
 U 1 1 5F550BB7
 P 8300 1400
@@
 $EndComp
 $Comp
-L GND #PWR05
+L power:GND #PWR05
 U 1 1 5F550C57
 P 8750 1550
@@
 $EndComp
 $Comp
-L BSS138 Q2
+L transistors:BSS138 Q2
 U 1 1 5F550E2F
 P 8650 2050
@@
 $EndComp
 $Comp
-L R R4
+L Device:R R4
 U 1 1 5F550E35
 P 8300 2200
@@
 $EndComp
 $Comp
-L GND #PWR06
+L power:GND #PWR06
 U 1 1 5F550E3B
 P 8750 2350
@@
 $EndComp
 $Comp
-L BSS138 Q3
+L transistors:BSS138 Q3
 U 1 1 5F550F8F
 P 8650 2850
@@
 $EndComp
 $Comp
-L R R5
+L Device:R R5
 U 1 1 5F550F95
 P 8300 3000
@@
 $EndComp
 $Comp
-L GND #PWR07
+L power:GND #PWR07
 U 1 1 5F550F9B
 P 8750 3150
@@
 $EndComp
 $Comp
-L Conn_01x04 J6
+L conn:Conn_01x04 J6
 U 1 1 5F551747
 P 9550 1050
@@
 $EndComp
 $Comp
-L +12V #PWR08
+L power:+12V #PWR08
 U 1 1 5F551831
 P 9350 1450
@@
 $EndComp
 $Comp
-L +12V #PWR09
+L power:+12V #PWR09
 U 1 1 5F551D85
 P 7050 4500
@@
 $EndComp
 $Comp
-L LM7805_TO220 U2
+L regul:LM7805_TO220 U2
 U 1 1 5F552340
 P 8500 4500
@@
 $EndComp
 $Comp
-L CP C6
+L Device:CP C6
 U 1 1 5F552FE1
 P 7850 4650
@@
 $EndComp
 $Comp
-L CP C7
+L Device:CP C7
 U 1 1 5F553050
 P 9150 4650
@@
 $EndComp
 $Comp
-L GND #PWR010
+L power:GND #PWR010
 U 1 1 5F55362D
 P 8500 4800
@@
 $EndComp
 $Comp
-L +5V #PWR011
+L power:+5V #PWR011
 U 1 1 5F553659
 P 9150 4500
@@
 $EndComp
 $Comp
-L Conn_01x02 J4
+L conn:Conn_01x02 J4
 U 1 1 5F5552F7
 P 3950 3350
@@
 $EndComp
 $Comp
-L +5V #PWR012
+L power:+5V #PWR012
 U 1 1 5F5553B3
 P 3650 3150
@@
 $EndComp
 $Comp
-L C C3
+L Device:C C3
 U 1 1 5F555F6E
 P 4050 3600
@@
 $EndComp
 $Comp
-L C C5
+L Device:C C5
 U 1 1 5F556003
 P 6050 3150
@@
 $EndComp
 $Comp
-L C C4
+L Device:C C4
 U 1 1 5F5560AE
 P 6050 2250
@@
 $EndComp
 $Comp
-L C C2
+L Device:C C2
 U 1 1 5F5564B5
 P 3650 2750
@@
 $EndComp
 $Comp
-L GND #PWR013
+L power:GND #PWR013
 U 1 1 5F5573B3
 P 4050 3750
@@
 $EndComp
 $Comp
-L Conn_01x03 J1
+L conn:Conn_01x03 J1
 U 1 1 5F561BA9
 P 1300 750
@@
 $EndComp
 $Comp
-L Conn_01x03 J2
+L conn:Conn_01x03 J2
 U 1 1 5F561C44
 P 1300 1350
@@
 $EndComp
 $Comp
-L Conn_01x03 J3
+L conn:Conn_01x03 J3
 U 1 1 5F561CC5
 P 1300 1900
@@
 $EndComp
 $Comp
-L GND #PWR014
+L power:GND #PWR014
 U 1 1 5F561D2B
 P 1500 1800
@@
 $EndComp
 $Comp
-L GND #PWR015
+L power:GND #PWR015
 U 1 1 5F561D72
 P 1500 1250
@@
 $EndComp
 $Comp
-L GND #PWR016
+L power:GND #PWR016
 U 1 1 5F561E1D
 P 1500 650
@@
 $EndComp
 $Comp
-L D D2
+L Device:D D2
 U 1 1 5F5637F2
 P 1850 1450
@@
 $EndComp
 $Comp
-L D D3
+L Device:D D3
 U 1 1 5F5638CA
 P 1850 2000
@@
 $EndComp
 $Comp
-L D D1
+L Device:D D1
 U 1 1 5F563940
 P 1850 850
@@
 $EndComp
 $Comp
-L R R1
+L Device:R R1
 U 1 1 5F563B4A
 P 2550 1500
@@
 $EndComp
 $Comp
-L R R2
+L Device:R R2
 U 1 1 5F563BC3
 P 2550 1800
@@
 $EndComp
 $Comp
-L GND #PWR017
+L power:GND #PWR017
 U 1 1 5F563C1D
 P 2550 1950
@@
 $EndComp
 $Comp
-L C C1
+L Device:C C1
 U 1 1 5F563D45
 P 3050 1800
@@
 B
 $Comp
-L CP C8
+L Device:CP C8
 U 1 1 5FB1AC4E
 P 3250 2850
@@
 $EndComp
 $Comp
-L +5V #PWR018
+L power:+5V #PWR018
 U 1 1 5FD4F943
 P 1500 750
@@
 $EndComp
 $Comp
-L +5V #PWR019
+L power:+5V #PWR019
 U 1 1 5FD4FC42
 P 1500 1350
@@
 $EndComp
 $Comp
-L +5V #PWR020
+L power:+5V #PWR020
 U 1 1 5FD4FC9E
 P 1500 1900
@@
 $EndComp
 $Comp
-L Screw_Terminal_01x02 J5
+L conn:Screw_Terminal_01x02 J5
 U 1 1 5FD50EFF
 P 6700 4600
@@
 $EndComp
 Wire Wire Line
-	7700 1250 8450 1250
+	7700 1250 8300 1250
 Wire Wire Line
 	8300 1550 8750 1550
@@
 	8750 1550 8750 1450
 Wire Wire Line
-	7800 2050 8450 2050
+	7800 2050 8300 2050
 Wire Wire Line
 	8300 2350 8750 2350
@@
 	5650 2350 6200 2350
 Wire Wire Line
-	5650 3050 6300 3050
+	5650 3050 6200 3050
 Wire Wire Line
 	5650 2450 7800 2450
@@
 Connection ~ 8750 1550
 Wire Wire Line
-	6900 4500 8200 4500
-Wire Wire Line
-	6900 4600 6900 4800
-Connection ~ 6900 4700
+	6900 4500 7050 4500
 Connection ~ 7050 4500
 Wire Wire Line
-	6900 4800 9150 4800
+	6900 4800 7850 4800
 Connection ~ 7850 4800
 Connection ~ 8500 4800
@@
 Connection ~ 9150 4500
 Wire Wire Line
-	3000 2650 4050 2650
+	3000 2650 3100 2650
 Wire Wire Line
 	4050 3150 3950 3150
@@
 	2000 1350 2550 1350
 Wire Wire Line
-	2550 1650 3250 1650
+	2550 1650 3050 1650
 Wire Wire Line
 	3250 1650 3250 1400
@@
 	1500 850  1700 850
 Wire Wire Line
-	2000 850  2000 2000
+	2000 850  2000 1350
 Connection ~ 2000 1450
 Wire Wire Line
@@
 Wire Wire Line
 	1700 2000 1500 2000
+Wire Wire Line
+	8300 1250 8450 1250
+Wire Wire Line
+	8300 2050 8450 2050
+Wire Wire Line
+	7050 4500 7850 4500
+Wire Wire Line
+	7850 4800 8500 4800
+Wire Wire Line
+	8500 4800 9150 4800
+Wire Wire Line
+	3500 2650 4050 2650
+Wire Wire Line
+	6200 3050 6300 3050
+Wire Wire Line
+	2000 1350 2000 1450
+Wire Wire Line
+	3050 1650 3250 1650
+Wire Wire Line
+	7850 4500 8200 4500
+Wire Wire Line
+	3100 2650 3500 2650
+Wire Wire Line
+	2000 1450 2000 2000
+Wire Wire Line
+	6900 4600 6900 4800
 $EndSCHEMATC
